File: Pulse_Box_PCB.kicad_pcb (KiCad board)
At the start: 2 copper layers, 40 x 50 mm, 35 parts, among them J1 Barrel_Jack, J2 Conn_02x05_Odd_Even, J3 USB_B_Micro, J4 Conn_01x03_Pin, U1 STM32F407VGTx, U2 SN74LV1T34DBV, U3 AP2112K-3.3, U4 TPSM53604RDA, Y1 8MHz Crystal

Commit message: organize schematic into power and signal pages, fixed wire nests
Parts:
- R1: value 10k -> 100k
- R2: value 2.37k -> 100k
- R3: value 100k -> 10k
- R4: value 100k -> 2.37k
Connections:
- net Net-(J2-RESET) renamed NRST
- net Net-(J2-SWDCLK) renamed SWDCLK
- net Net-(J2-SWDIO) renamed SWDIO
- net Net-(J2-SWO) renamed SWO
- net Net-(J2-UART_RX) renamed UART_RX
- net Net-(J2-UART_TX) renamed UART_TX
- net Net-(J3-D+) renamed USB_DP
- net Net-(J3-D-) renamed USB_DM
- net Net-(J3-VBUS) renamed VBUS
- net Net-(J4-Pin_2) renamed PWM_5V5
- net Net-(U1-PA7) renamed PWM_3V3
- C13 pad 1: +3.3V -> GND
- C13 pad 2: GND -> +3.3V
- C19 pad 1: +3.3V -> GND
- C19 pad 2: GND -> +3.3V
- C20 pad 2: +3.3V -> Net-(U1-VDDA)
- C21 pad 1: +3.3V -> Net-(U1-VDDA)
- C8 pad 1: +3.3V -> GND
- C8 pad 2: GND -> +3.3V
- R1 pad 1: +5V -> +24V
- R1 pad 2: Net-(U4-FB) -> Net-(U4-EN)
- R2 pad 1: Net-(U4-FB) -> Net-(U4-V5V)
- R2 pad 2: GND -> Net-(U4-PGOOD)
- R3 pad 1: Net-(U4-V5V) -> +5V
- R3 pad 2: Net-(U4-PGOOD) -> Net-(U4-FB)
- R4 pad 1: +24V -> Net-(U4-FB)
- R4 pad 2: Net-(U4-EN) -> GND
- U1 pad 22: +3.3V -> Net-(U1-VDDA)
Routing:
- net GND: track 43.2 -> 41.3 mm, vias 10 -> 9
- net +3.3V: track 115.2 -> 117.0 mm, vias 6 -> 7
