File: Pulse_Box_PCB_v2/power.kicad_sch (KiCad schematic)
At the start: 31 parts, among them J1 Screw_Terminal_01x02, J7 Conn_01x04, U3 TPS54560BDDA, U5 74LVC1G3157, U8 AP2114-3.3TRG1

Commit message: v2 board mirrored layout
Connections:
- net +24V: now also J1.1 (Pin_1); no longer J1.2 (Pin_2)
- net GND: now also J1.2 (Pin_2); no longer J1.1 (Pin_1)
Other:
- moved on the sheet: C1
Changed lines of the file:
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@@
 	)
 	(junction
+		(at 54.61 52.07)
+		(diameter 0)
+		(color 0 0 0 0)
+	)
+	(junction
 		(at 43.18 124.46)
 		(diameter 0)
@@
 	)
 	(junction
-		(at 54.61 52.07)
-		(diameter 0)
-		(color 0 0 0 0)
-	)
-	(junction
 		(at 140.97 82.55)
 		(diameter 0)
@@
 	)
 	(junction
-		(at 54.61 72.39)
-		(diameter 0)
-		(color 0 0 0 0)
-	)
-	(junction
 		(at 43.18 149.86)
 		(diameter 0)
@@
 	)
 	(junction
+		(at 54.61 72.39)
+		(diameter 0)
+		(color 0 0 0 0)
+	)
+	(junction
 		(at 213.36 87.63)
 		(diameter 0)
@@
 	(wire
 		(pts
+			(xy 59.69 45.72) (xy 54.61 45.72)
+		)
+		(stroke
+			(width 0)
+			(type default)
+		)
+	)
+	(wire
+		(pts
 			(xy 140.97 140.97) (xy 140.97 148.59)
 		)
@@
 	(wire
 		(pts
+			(xy 60.96 80.01) (xy 54.61 80.01)
+		)
+		(stroke
+			(width 0)
+			(type default)
+		)
+	)
+	(wire
+		(pts
 			(xy 115.57 54.61) (xy 115.57 36.83)
 		)
@@
 	(wire
 		(pts
+			(xy 54.61 80.01) (xy 54.61 72.39)
+		)
+		(stroke
+			(width 0)
+			(type default)
+		)
+	)
+	(wire
+		(pts
 			(xy 157.48 62.23) (xy 157.48 71.12)
 		)
@@
 	(wire
 		(pts
-			(xy 140.97 54.61) (xy 132.08 54.61)
+			(xy 54.61 45.72) (xy 54.61 52.07)
 		)
 		(stroke
@@
 	(wire
 		(pts
-			(xy 81.28 176.53) (xy 74.93 176.53)
+			(xy 140.97 54.61) (xy 132.08 54.61)
 		)
 		(stroke
@@
 	(wire
 		(pts
-			(xy 140.97 148.59) (xy 125.73 148.59)
+			(xy 81.28 176.53) (xy 74.93 176.53)
 		)
 		(stroke
@@
 	(wire
 		(pts
-			(xy 54.61 72.39) (xy 54.61 76.2)
+			(xy 140.97 148.59) (xy 125.73 148.59)
 		)
 		(stroke
@@
 	(wire
 		(pts
-			(xy 54.61 52.07) (xy 54.61 46.99)
-		)
-		(stroke
-			(width 0)
-			(type default)
-		)
-	)
-	(wire
-		(pts
 			(xy 68.58 173.99) (xy 68.58 171.45)
 		)
@@
 	(symbol
 		(lib_id "power:GND")
-		(at 54.61 76.2 0)
+		(at 59.69 45.72 0)
 		(unit 1)
 		(exclude_from_sim no)
@@
 		(fields_autoplaced yes)
 		(property "Reference" "#PWR018"
-			(at 54.61 82.55 0)
+			(at 59.69 52.07 0)
 			(effects
 				(font
@@
 		)
 		(property "Value" "GND"
-			(at 54.61 81.28 0)
+			(at 59.69 50.8 0)
 			(effects
 				(font
@@
 		)
 		(property "Footprint" ""
-			(at 54.61 76.2 0)
+			(at 59.69 45.72 0)
 			(effects
 				(font
@@
 		)
 		(property "Datasheet" ""
-			(at 54.61 76.2 0)
+			(at 59.69 45.72 0)
 			(effects
 				(font
@@
 		)
 		(property "Description" "Power symbol creates a global label with name \"GND\" , ground"
-			(at 54.61 76.2 0)
+			(at 59.69 45.72 0)
 			(effects
 				(font
@@
 	(symbol
 		(lib_id "power:+24V")
-		(at 54.61 46.99 0)
+		(at 60.96 80.01 0)
 		(unit 1)
 		(exclude_from_sim no)
@@
 		(fields_autoplaced yes)
 		(property "Reference" "#PWR017"
-			(at 54.61 50.8 0)
+			(at 60.96 83.82 0)
 			(effects
 				(font
@@
 		)
 		(property "Value" "+24V"
-			(at 54.61 41.91 0)
+			(at 60.96 74.93 0)
 			(effects
 				(font
@@
 		)
 		(property "Footprint" ""
-			(at 54.61 46.99 0)
+			(at 60.96 80.01 0)
 			(effects
 				(font
@@
 		)
 		(property "Datasheet" ""
-			(at 54.61 46.99 0)
+			(at 60.96 80.01 0)
 			(effects
 				(font
@@
 		)
 		(property "Description" "Power symbol creates a global label with name \"+24V\""
-			(at 54.61 46.99 0)
+			(at 60.96 80.01 0)
 			(effects
 				(font
@@
 	(symbol
 		(lib_id "Device:C_Polarized_US")
-		(at 64.77 62.23 0)
+		(at 64.77 62.23 180)
 		(unit 1)
 		(exclude_from_sim no)
@@
 		(dnp no)
 		(property "Reference" "C1"
-			(at 68.58 61.214 0)
+			(at 60.96 63.246 0)
 			(effects
 				(font
@@
 		)
 		(property "Value" "470uF"
-			(at 68.58 63.754 0)
+			(at 60.96 60.706 0)
 			(effects
 				(font
