File: Pulse_Box_PCB_v2/signals.kicad_sch (KiCad schematic)
At the start: 31 parts

Commit message: add design for pulsebox panel, update v2 PCB to remove 485 trans
Parts:
- removed C?: 100nF, Capacitor_SMD:C_0402_1005Metric, symbol Device:C
- removed D?: SP0502BAHT, Package_TO_SOT_SMD:SOT-23, symbol Power_Protection:SP0502BAHT
- removed R?: 120, Resistor_SMD:R_0402_1005Metric, symbol Device:R
- removed TP?: TestPoint, TestPoint:TestPoint_Pad_2.0x2.0mm, symbol Connector:TestPoint
- removed U?: SP3485EN, Package_SO:SOIC-8_3.9x4.9mm_P1.27mm, symbol Interface_UART:SP3485EN
- added C15: 100nF, Capacitor_SMD:C_0402_1005Metric, symbol Device:C
- added R14, R5: 22, Resistor_SMD:R_0402_1005Metric, symbol Device:R
- added U4: SN74LV1T34DBV, Package_TO_SOT_SMD:SOT-23-5, symbol Logic_LevelTranslator:SN74LV1T34DBV
- R7, R8: renamed from R?; value 47k -> 10k; JLCPCB Part # C25792 -> C25744
- U5: renamed from U?; JLCPCB Part # C52140494 -> C10426
- gave numbers to parts that had none: 23
Connections:
- net 485_DE is gone; now on net UART1_TX: U1.32 (IO39)
- net +5V: now also C15.1, U4.5 (VCC)
- net DM: now also R14.1; no longer U2.3 (I/O2)
- net DP: now also R5.1; no longer U2.1 (I/O1)
- net E_SENS: now also U1.35 (IO42); no longer U1.39 (IO1)
- net GND: now also C15.2, U4.3 (GND)
- net PWM_SEL: now also U4.2 (A); no longer U5.6
- net UART1_RX: now also J3.8 (Pin_8)
- net UART1_TX: now also J3.4 (Pin_4); no longer U1.31 (IO38)
- net UART2_TX: now reaches U1.24 (IO47)
- net UART2_TX: now also J2.4 (Pin_4)
- net UART2_RX: now reaches U1.25 (IO48)
- net UART2_RX: now also J2.8 (Pin_8)
- removed net 485A: J2.4 (Pin_4), J2.8 (Pin_8), J3.4 (Pin_4), J3.8 (Pin_8)
- removed net 485B: J2.5 (Pin_5), J2.7 (Pin_7), J3.5 (Pin_5), J3.7 (Pin_7)
- new net: U4.4 (Y), U5.6
- new net: R5.2, U2.1 (I/O1)
- new net: R14.2, U2.3 (I/O2)
Other:
- moved on the sheet: D3, D4, J2, J3, J4, J5, R10, R11, R12, R7, R8, U5A

Commit message: v2 board mirrored layout
Parts:
- J4, J5: footprint Connector_JST:JST_PH_S3B-PH-SM4-TB_1x03-1MP_P2.00mm_Horizontal -> Connector_JST:JST_PH_B3B-PH-K_1x03_P2.00mm_Vertical
Connections:
- net E_SENS: now also U1.11 (IO18); no longer U1.35 (IO42)
- net UART1_RX: now also U1.10 (IO17); no longer U1.33 (IO40)
- net UART1_TX: now also U1.9 (IO16); no longer U1.32 (IO39)
- net UART2_RX: now also U1.24 (IO47); no longer U1.25 (IO48)
- net UART2_TX: now also U1.23 (IO21); no longer U1.24 (IO47)
- net S_SENS renamed N_SENS
- net N_SENS: now also U1.25 (IO48); no longer U1.22 (IO14)
Changed lines of the file:
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@@
 	(wire
 		(pts
+			(xy 93.98 57.15) (xy 99.06 57.15)
+		)
+		(stroke
+			(width 0)
+			(type default)
+		)
+	)
+	(wire
+		(pts
 			(xy 255.27 137.16) (xy 255.27 139.7)
 		)
@@
 	(wire
 		(pts
-			(xy 17.78 119.38) (xy 17.78 124.46)
+			(xy 59.69 95.25) (xy 63.5 95.25)
 		)
 		(stroke
@@
 	(wire
 		(pts
-			(xy 213.36 125.73) (xy 241.3 125.73)
+			(xy 17.78 119.38) (xy 17.78 124.46)
 		)
 		(stroke
@@
 	(wire
 		(pts
-			(xy 78.74 20.32) (xy 78.74 31.75)
+			(xy 213.36 125.73) (xy 241.3 125.73)
 		)
 		(stroke
@@
 	(wire
 		(pts
-			(xy 93.98 92.71) (xy 99.06 92.71)
+			(xy 78.74 20.32) (xy 78.74 31.75)
 		)
 		(stroke
@@
 	(wire
 		(pts
+			(xy 93.98 95.25) (xy 99.06 95.25)
+		)
+		(stroke
+			(width 0)
+			(type default)
+		)
+	)
+	(wire
+		(pts
 			(xy 222.25 58.42) (xy 222.25 57.15)
 		)
@@
 	(wire
 		(pts
-			(xy 93.98 77.47) (xy 99.06 77.47)
-		)
-		(stroke
-			(width 0)
-			(type default)
-		)
-	)
-	(wire
-		(pts
 			(xy 172.72 133.35) (xy 182.88 133.35)
 		)
@@
 	(wire
 		(pts
-			(xy 93.98 85.09) (xy 99.06 85.09)
-		)
-		(stroke
-			(width 0)
-			(type default)
-		)
-	)
-	(wire
-		(pts
 			(xy 222.25 71.12) (xy 214.63 71.12)
 		)
@@
 	(wire
 		(pts
+			(xy 93.98 64.77) (xy 99.06 64.77)
+		)
+		(stroke
+			(width 0)
+			(type default)
+		)
+	)
+	(wire
+		(pts
 			(xy 184.15 95.25) (xy 189.23 95.25)
 		)
@@
 	(wire
 		(pts
-			(xy 59.69 90.17) (xy 63.5 90.17)
-		)
-		(stroke
-			(width 0)
-			(type default)
-		)
-	)
-	(wire
-		(pts
 			(xy 222.25 57.15) (xy 231.14 57.15)
 		)
@@
 	(wire
 		(pts
-			(xy 219.71 74.93) (xy 219.71 82.55)
+			(xy 93.98 92.71) (xy 99.06 92.71)
 		)
 		(stroke
@@
 	(wire
 		(pts
-			(xy 78.74 38.1) (xy 87.63 38.1)
+			(xy 219.71 74.93) (xy 219.71 82.55)
 		)
 		(stroke
@@
 	(wire
 		(pts
-			(xy 241.3 146.05) (xy 241.3 156.21)
+			(xy 93.98 54.61) (xy 99.06 54.61)
 		)
 		(stroke
@@
 	(wire
 		(pts
-			(xy 17.78 107.95) (xy 17.78 119.38)
+			(xy 78.74 38.1) (xy 87.63 38.1)
 		)
 		(stroke
@@
 	(wire
 		(pts
-			(xy 182.88 143.51) (xy 154.94 143.51)
+			(xy 241.3 146.05) (xy 241.3 156.21)
 		)
 		(stroke
@@
 	(wire
 		(pts
-			(xy 80.01 137.16) (xy 74.93 137.16)
+			(xy 17.78 107.95) (xy 17.78 119.38)
 		)
 		(stroke
@@
 	(wire
 		(pts
-			(xy 184.15 55.88) (xy 184.15 62.23)
+			(xy 182.88 143.51) (xy 154.94 143.51)
 		)
 		(stroke
@@
 	(wire
 		(pts
-			(xy 74.93 137.16) (xy 74.93 139.7)
+			(xy 80.01 137.16) (xy 74.93 137.16)
 		)
 		(stroke
@@
 	(wire
 		(pts
-			(xy 127 45.72) (xy 127 50.8)
+			(xy 184.15 55.88) (xy 184.15 62.23)
 		)
 		(stroke
@@
 	(wire
 		(pts
-			(xy 36.83 46.99) (xy 36.83 49.53)
+			(xy 74.93 137.16) (xy 74.93 139.7)
 		)
 		(stroke
@@
 	(wire
 		(pts
-			(xy 93.98 95.25) (xy 99.06 95.25)
+			(xy 127 45.72) (xy 127 50.8)
 		)
 		(stroke
@@
 	(wire
 		(pts
-			(xy 120.65 90.17) (xy 120.65 95.25)
+			(xy 36.83 46.99) (xy 36.83 49.53)
 		)
 		(stroke
@@
 	(wire
 		(pts
-			(xy 182.88 156.21) (xy 166.37 156.21)
+			(xy 120.65 90.17) (xy 120.65 95.25)
 		)
 		(stroke
@@
 	(wire
 		(pts
-			(xy 214.63 71.12) (xy 214.63 92.71)
+			(xy 182.88 156.21) (xy 166.37 156.21)
 		)
 		(stroke
@@
 	(wire
 		(pts
-			(xy 93.98 80.01) (xy 99.06 80.01)
+			(xy 214.63 71.12) (xy 214.63 92.71)
 		)
 		(stroke
@@
 	(global_label "UART2_TX"
 		(shape input)
-		(at 99.06 92.71 0)
+		(at 99.06 64.77 0)
 		(fields_autoplaced yes)
 		(effects
@@
 		)
 		(property "Intersheetrefs" "${INTERSHEET_REFS}"
-			(at 111.0561 92.71 0)
+			(at 111.0561 64.77 0)
 			(effects
 				(font
@@
 		)
 	)
-	(global_label "S_SENS"
+	(global_label "N_SENS"
 		(shape input)
-		(at 59.69 90.17 180)
+		(at 99.06 95.25 0)
 		(fields_autoplaced yes)
 		(effects
@@
 				(size 1.27 1.27)
 			)
-			(justify right)
+			(justify left)
 		)
 		(property "Intersheetrefs" "${INTERSHEET_REFS}"
-			(at 49.6292 90.17 0)
+			(at 109.2418 95.25 0)
 			(effects
 				(font
 					(size 1.27 1.27)
 				)
-				(justify right)
+				(justify left)
 				(hide yes)
 			)
 		)
 	)
-	(global_label "S_SENS"
+	(global_label "N_SENS"
 		(shape input)
 		(at 255.27 139.7 270)
@@
 		)
 		(property "Intersheetrefs" "${INTERSHEET_REFS}"
-			(at 255.27 149.7608 90)
+			(at 255.27 149.8818 90)
 			(effects
 				(font
@@
 	(global_label "UART2_RX"
 		(shape input)
-		(at 99.06 95.25 0)
+		(at 99.06 92.71 0)
 		(fields_autoplaced yes)
 		(effects
@@
 		)
 		(property "Intersheetrefs" "${INTERSHEET_REFS}"
-			(at 111.3585 95.25 0)
+			(at 111.3585 92.71 0)
 			(effects
 				(font
@@
 	(global_label "UART1_TX"
 		(shape input)
-		(at 99.06 77.47 0)
+		(at 59.69 95.25 180)
 		(fields_autoplaced yes)
 		(effects
@@
 				(size 1.27 1.27)
 			)
-			(justify left)
+			(justify right)
 		)
 		(property "Intersheetrefs" "${INTERSHEET_REFS}"
-			(at 111.0561 77.47 0)
+			(at 47.6939 95.25 0)
 			(effects
 				(font
 					(size 1.27 1.27)
 				)
-				(justify left)
+				(justify right)
 				(hide yes)
 			)
@@
 	(global_label "E_SENS"
 		(shape input)
-		(at 99.06 85.09 0)
+		(at 99.06 57.15 0)
 		(fields_autoplaced yes)
 		(effects
@@
 		)
 		(property "Intersheetrefs" "${INTERSHEET_REFS}"
-			(at 109.0603 85.09 0)
+			(at 109.0603 57.15 0)
 			(effects
 				(font
@@
 		)
 	)
-	(global_label "S_SENS"
+	(global_label "N_SENS"
 		(shape input)
 		(at 231.14 140.97 180)
@@
 		)
 		(property "Intersheetrefs" "${INTERSHEET_REFS}"
-			(at 221.0792 140.97 0)
+			(at 220.9582 140.97 0)
 			(effects
 				(font
@@
 	(global_label "UART1_RX"
 		(shape input)
-		(at 99.06 80.01 0)
+		(at 99.06 54.61 0)
 		(fields_autoplaced yes)
 		(effects
@@
 		)
 		(property "Intersheetrefs" "${INTERSHEET_REFS}"
-			(at 111.3585 80.01 0)
+			(at 111.3585 54.61 0)
 			(effects
 				(font
@@
 			)
 		)
-		(property "Footprint" "Connector_JST:JST_PH_S3B-PH-SM4-TB_1x03-1MP_P2.00mm_Horizontal"
+		(property "Footprint" "Connector_JST:JST_PH_B3B-PH-K_1x03_P2.00mm_Vertical"
 			(at 85.09 160.02 0)
 			(effects
@@
 			)
 		)
-		(property "Footprint" "Connector_JST:JST_PH_S3B-PH-SM4-TB_1x03-1MP_P2.00mm_Horizontal"
+		(property "Footprint" "Connector_JST:JST_PH_B3B-PH-K_1x03_P2.00mm_Vertical"
 			(at 85.09 134.62 0)
 			(effects
