File: Pulse_Box_Panel_v1/power.kicad_sch (KiCad schematic)
At the start: 19 parts, among them J9 Conn_01x04_Pin, U4 TPS54560BDDA, U5 AP2112K-3.3

Commit message: complete v2 and v1 panel design, this is the final design sent to jlcpcb for v2
Parts:
- added H1, H2, H3, H4: MountingHole, MountingHole:MountingHole_3.2mm_M3, symbol Mechanical:MountingHole
- L1: footprint Inductor_SMD:L_APV_APH1030 -> Inductor_SMD:L_TechFuse_SL1040
- U3: renamed from U5; JLCPCB Part # C51118 -> C3021085
- renumbered C3 to C1, C19 to C10, C4 to C2, C5 to C3, C6 to C4, C7 to C5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
