File: Pulse_Box_Panel_v1/signals.kicad_sch (KiCad schematic)
At the start: 25 parts, among them J1 Conn_01x11, J2 Conn_01x11, J3 Conn_01x11, J4 Conn_01x11, J5 Conn_01x03, J6 Conn_01x03, J7 Conn_02x05_Odd_Even, J8 Conn_01x03, U1 STM32G0B1CBTx, U2 74HCT4051, U3 74HCT4051, Y1 8MHz Crystal

Commit message: complete v2 and v1 panel design, this is the final design sent to jlcpcb for v2
Parts:
- J5, J6: footprint Connector_JST:JST_PH_S3B-PH-SM4-TB_1x03-1MP_P2.00mm_Horizontal -> Connector_JST:JST_PH_B3B-PH-K_1x03_P2.00mm_Vertical; JLCPCB Part # C265101 -> C131339
- renumbered C2 to C11, C1 to C12, C18 to C16, C16 to C18, C20 to C19, J4 to J1, J3 to J2, J1 to J3, J2 to J4, J7 to J9, U3 to U4, U2 to U5
Connections:
- net E_LED_PWM: now also J1.6 (Pin_6), U4.12 (A3), U5.15 (A2); no longer J3.6 (Pin_6), U4.15 (A2), U5.12 (A3)
- net W_LED_PWM: now also J3.6 (Pin_6), U4.15 (A2), U5.12 (A3); no longer J1.6 (Pin_6), U4.12 (A3), U5.15 (A2)
Changed lines of the file:
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@@
 		)
 	)
+	(global_label "E_LED_PWM"
+		(shape input)
+		(at 215.9 121.92 180)
+		(fields_autoplaced yes)
+		(effects
+			(font
+				(size 1.27 1.27)
+			)
+			(justify right)
+		)
+		(property "Intersheetrefs" "${INTERSHEET_REFS}"
+			(at 202.2107 121.92 0)
+			(effects
+				(font
+					(size 1.27 1.27)
+				)
+				(justify right)
+				(hide yes)
+			)
+		)
+	)
 	(global_label "UART3_RX"
 		(shape input)
@@
 		)
 	)
-	(global_label "W_LED_PWM"
+	(global_label "E_LED_PWM"
 		(shape input)
-		(at 172.72 110.49 0)
+		(at 175.26 161.29 0)
 		(fields_autoplaced yes)
 		(effects
@@
 		)
 		(property "Intersheetrefs" "${INTERSHEET_REFS}"
-			(at 186.7117 110.49 0)
+			(at 188.9493 161.29 0)
 			(effects
 				(font
@@
 		)
 	)
-	(global_label "E_LED_PWM"
+	(global_label "MUX_IN_S0"
 		(shape input)
-		(at 175.26 158.75 0)
+		(at 146.05 110.49 180)
 		(fields_autoplaced yes)
 		(effects
@@
 				(size 1.27 1.27)
 			)
-			(justify left)
+			(justify right)
 		)
 		(property "Intersheetrefs" "${INTERSHEET_REFS}"
-			(at 188.9493 158.75 0)
+			(at 132.7839 110.49 0)
 			(effects
 				(font
 					(size 1.27 1.27)
 				)
-				(justify left)
+				(justify right)
 				(hide yes)
 			)
 		)
 	)
-	(global_label "MUX_IN_S0"
+	(global_label "W_LED_PWM"
 		(shape input)
-		(at 146.05 110.49 180)
+		(at 172.72 113.03 0)
 		(fields_autoplaced yes)
 		(effects
@@
 				(size 1.27 1.27)
 			)
-			(justify right)
+			(justify left)
 		)
 		(property "Intersheetrefs" "${INTERSHEET_REFS}"
-			(at 132.7839 110.49 0)
+			(at 186.7117 113.03 0)
 			(effects
 				(font
 					(size 1.27 1.27)
 				)
-				(justify right)
+				(justify left)
 				(hide yes)
 			)
@@
 		)
 	)
-	(global_label "UART1_TX"
+	(global_label "E_LED_PWM"
 		(shape input)
-		(at 100.33 86.36 0)
+		(at 172.72 110.49 0)
 		(fields_autoplaced yes)
 		(effects
@@
 		)
 		(property "Intersheetrefs" "${INTERSHEET_REFS}"
-			(at 112.3261 86.36 0)
+			(at 186.4093 110.49 0)
 			(effects
 				(font
@@
 		)
 	)
-	(global_label "E_LED_PWM"
+	(global_label "UART1_TX"
 		(shape input)
-		(at 261.62 119.38 180)
+		(at 100.33 86.36 0)
 		(fields_autoplaced yes)
 		(effects
@@
 				(size 1.27 1.27)
 			)
-			(justify right)
+			(justify left)
 		)
 		(property "Intersheetrefs" "${INTERSHEET_REFS}"
-			(at 247.9307 119.38 0)
+			(at 112.3261 86.36 0)
 			(effects
 				(font
 					(size 1.27 1.27)
 				)
-				(justify right)
+				(justify left)
 				(hide yes)
 			)
@@
 		)
 	)
-	(global_label "W_LED_PWM"
-		(shape input)
-		(at 175.26 161.29 0)
-		(fields_autoplaced yes)
-		(effects
-			(font
-				(size 1.27 1.27)
-			)
-			(justify left)
-		)
-		(property "Intersheetrefs" "${INTERSHEET_REFS}"
-			(at 189.2517 161.29 0)
-			(effects
-				(font
-					(size 1.27 1.27)
-				)
-				(justify left)
-				(hide yes)
-			)
-		)
-	)
 	(global_label "W_SENSE"
 		(shape input)
@@
 		)
 	)
-	(global_label "W_LED_PWM"
-		(shape input)
-		(at 215.9 121.92 180)
-		(fields_autoplaced yes)
-		(effects
-			(font
-				(size 1.27 1.27)
-			)
-			(justify right)
-		)
-		(property "Intersheetrefs" "${INTERSHEET_REFS}"
-			(at 201.9083 121.92 0)
-			(effects
-				(font
-					(size 1.27 1.27)
-				)
-				(justify right)
-				(hide yes)
-			)
-		)
-	)
 	(global_label "UART2_TX"
 		(shape input)
@@
 		)
 	)
+	(global_label "W_LED_PWM"
+		(shape input)
+		(at 261.62 119.38 180)
+		(fields_autoplaced yes)
+		(effects
+			(font
+				(size 1.27 1.27)
+			)
+			(justify right)
+		)
+		(property "Intersheetrefs" "${INTERSHEET_REFS}"
+			(at 247.6283 119.38 0)
+			(effects
+				(font
+					(size 1.27 1.27)
+				)
+				(justify right)
+				(hide yes)
+			)
+		)
+	)
 	(global_label "E_SENSE"
 		(shape input)
@@
 		)
 	)
-	(global_label "E_LED_PWM"
-		(shape input)
-		(at 172.72 113.03 0)
-		(fields_autoplaced yes)
-		(effects
-			(font
-				(size 1.27 1.27)
-			)
-			(justify left)
-		)
-		(property "Intersheetrefs" "${INTERSHEET_REFS}"
-			(at 186.4093 113.03 0)
-			(effects
-				(font
-					(size 1.27 1.27)
-				)
-				(justify left)
-				(hide yes)
-			)
-		)
-	)
 	(global_label "S_LED_PWM"
 		(shape input)
@@
 		)
 	)
+	(global_label "W_LED_PWM"
+		(shape input)
+		(at 175.26 158.75 0)
+		(fields_autoplaced yes)
+		(effects
+			(font
+				(size 1.27 1.27)
+			)
+			(justify left)
+		)
+		(property "Intersheetrefs" "${INTERSHEET_REFS}"
+			(at 189.2517 158.75 0)
+			(effects
+				(font
+					(size 1.27 1.27)
+				)
+				(justify left)
+				(hide yes)
+			)
+		)
+	)
 	(symbol
 		(lib_id "power:+24V")
@@
 		(dnp no)
 		(fields_autoplaced yes)
-		(property "Reference" "C16"
+		(property "Reference" "C18"
 			(at 229.87 149.2249 0)
 			(effects
@@
 			(project ""
 				(path "/4517addf-2697-4ea8-8228-462c8f611da2/df59875f-eeef-414a-8ccd-577ddbc838a1"
-					(reference "C16")
+					(reference "C18")
 					(unit 1)
 				)
@@
 		(on_board yes)
 		(dnp no)
-		(property "Reference" "J2"
+		(property "Reference" "J4"
 			(at 193.294 26.162 0)
 			(effects
@@
 			(project "Pulse_Box_Panel_v1"
 				(path "/4517addf-2697-4ea8-8228-462c8f611da2/df59875f-eeef-414a-8ccd-577ddbc838a1"
-					(reference "J2")
+					(reference "J4")
 					(unit 1)
 				)
@@
 		(dnp no)
 		(fields_autoplaced yes)
-		(property "Reference" "U3"
+		(property "Reference" "U4"
 			(at 162.1633 146.05 0)
 			(effects
@@
 			(project "Pulse_Box_Panel_v1"
 				(path "/4517addf-2697-4ea8-8228-462c8f611da2/df59875f-eeef-414a-8ccd-577ddbc838a1"
-					(reference "U3")
+					(reference "U4")
 					(unit 1)
 				)
@@
 		(on_board yes)
 		(dnp no)
-		(property "Reference" "J3"
+		(property "Reference" "J2"
 			(at 242.062 22.606 0)
 			(effects
@@
 			(project "Pulse_Box_Panel_v1"
 				(path "/4517addf-2697-4ea8-8228-462c8f611da2/df59875f-eeef-414a-8ccd-577ddbc838a1"
-					(reference "J3")
+					(reference "J2")
 					(unit 1)
 				)
@@
 		(on_board yes)
 		(dnp no)
-		(property "Reference" "C2"
+		(property "Reference" "C11"
 			(at 78.486 41.656 90)
 			(effects
@@
 			(project "Pulse_Box_Panel_v1"
 				(path "/4517addf-2697-4ea8-8228-462c8f611da2/df59875f-eeef-414a-8ccd-577ddbc838a1"
-					(reference "C2")
+					(reference "C11")
 					(unit 1)
 				)
@@
 		(dnp no)
 		(fields_autoplaced yes)
-		(property "Reference" "C20"
+		(property "Reference" "C19"
 			(at 274.32 73.0249 0)
 			(effects
@@
 			(project "Pulse_Box_Panel_v1"
 				(path "/4517addf-2697-4ea8-8228-462c8f611da2/df59875f-eeef-414a-8ccd-577ddbc838a1"
-					(reference "C20")
+					(reference "C19")
 					(unit 1)
 				)
@@
 			)
 		)
-		(property "Footprint" "Connector_JST:JST_PH_S3B-PH-SM4-TB_1x03-1MP_P2.00mm_Horizontal"
+		(property "Footprint" "Connector_JST:JST_PH_B3B-PH-K_1x03_P2.00mm_Vertical"
 			(at 163.83 38.1 0)
 			(effects
@@
 			)
 		)
-		(property "JLCPCB Part #" "C265101"
+		(property "JLCPCB Part #" "C131339"
 			(at 163.83 38.1 0)
 			(effects
@@
 			)
 		)
-		(property "Footprint" "Connector_JST:JST_PH_S3B-PH-SM4-TB_1x03-1MP_P2.00mm_Horizontal"
+		(property "Footprint" "Connector_JST:JST_PH_B3B-PH-K_1x03_P2.00mm_Vertical"
 			(at 163.83 63.5 0)
 			(effects
@@
 			)
 		)
-		(property "JLCPCB Part #" "C265101"
+		(property "JLCPCB Part #" "C131339"
 			(at 163.83 63.5 0)
 			(effects
@@
 		(dnp no)
 		(fields_autoplaced yes)
-		(property "Reference" "U2"
+		(property "Reference" "U5"
 			(at 159.6233 97.79 0)
 			(effects
@@
 			(project ""
 				(path "/4517addf-2697-4ea8-8228-462c8f611da2/df59875f-eeef-414a-8ccd-577ddbc838a1"
-					(reference "U2")
+					(reference "U5")
 					(unit 1)
 				)
@@
 		(on_board yes)
 		(dnp no)
-		(property "Reference" "C1"
+		(property "Reference" "C12"
 			(at 79.756 35.56 90)
 			(effects
@@
 			(project "Pulse_Box_Panel_v1"
 				(path "/4517addf-2697-4ea8-8228-462c8f611da2/df59875f-eeef-414a-8ccd-577ddbc838a1"
-					(reference "C1")
+					(reference "C12")
 					(unit 1)
 				)
@@
 		(on_board yes)
 		(dnp no)
-		(property "Reference" "J7"
+		(property "Reference" "J9"
 			(at 33.02 16.51 0)
 			(effects
@@
 			(project "Pulse_Box_Panel_v1"
 				(path "/4517addf-2697-4ea8-8228-462c8f611da2/df59875f-eeef-414a-8ccd-577ddbc838a1"
-					(reference "J7")
+					(reference "J9")
 					(unit 1)
 				)
@@
 		(on_board yes)
 		(dnp no)
-		(property "Reference" "C18"
+		(property "Reference" "C16"
 			(at 30.48 74.168 0)
 			(effects
@@
 			(project "Pulse_Box_Panel_v1"
 				(path "/4517addf-2697-4ea8-8228-462c8f611da2/df59875f-eeef-414a-8ccd-577ddbc838a1"
-					(reference "C18")
+					(reference "C16")
 					(unit 1)
 				)
@@
 		(on_board yes)
 		(dnp no)
-		(property "Reference" "J1"
+		(property "Reference" "J3"
 			(at 242.57 96.012 0)
 			(effects
@@
 			(project "Pulse_Box_Panel_v1"
 				(path "/4517addf-2697-4ea8-8228-462c8f611da2/df59875f-eeef-414a-8ccd-577ddbc838a1"
-					(reference "J1")
+					(reference "J3")
 					(unit 1)
 				)
@@
 		(on_board yes)
 		(dnp no)
-		(property "Reference" "J4"
+		(property "Reference" "J1"
 			(at 196.85 98.806 0)
 			(effects
@@
 			(project "Pulse_Box_Panel_v1"
 				(path "/4517addf-2697-4ea8-8228-462c8f611da2/df59875f-eeef-414a-8ccd-577ddbc838a1"
-					(reference "J4")
+					(reference "J1")
 					(unit 1)
 				)

Commit message: basic readme with board summaries
Connections:
- net E_SENSE: now also J1.9 (Pin_9), U1.43 (PB4); no longer J3.9 (Pin_9), U1.24 (PB12)
- net W_SENSE: now also J3.9 (Pin_9), U1.24 (PB12); no longer J1.9 (Pin_9), U1.43 (PB4)
